File: RSC-MBS-Backplane-28S-Lite.kicad_pcb (KiCad board)
At the start: 2 copper layers, 364 x 100 mm, 22 parts, among them J1 5530843-7, J10 5530843-7, J11 5530843-7, J12 5530843-7, J13 5530843-7, J14 5530843-7, J15 Conn_01x02, J16 Conn_02x08_Top_Bottom, J17 Conn_02x08_Top_Bottom, J18 Conn_01x02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

Commit message: initial attempt at routing balance traces
Parts:
- moved J15 414.7 mm to (109.3, 201.5), turned to 90 degrees
- moved J18 134.4 mm to (454.7, 198.5), turned to -90 degrees
- moved J17 0.13 mm to (454.7, 154.1)
Routing:
- net TAP8: track 0.00 -> 459.9 mm, vias 0 -> 1
- net TAP0: track 0.00 -> 442.8 mm
- net TAP14: track 0.00 -> 416.4 mm
- net TAP4: track 0.00 -> 407.6 mm, vias 0 -> 1
- net TAP2: track 0.00 -> 407.1 mm, vias 0 -> 1
- net TAP6: track 0.00 -> 403.4 mm, vias 0 -> 1
- net TAP10: track 0.00 -> 400.1 mm, vias 0 -> 1
- net TAP12: track 0.00 -> 398.3 mm, vias 0 -> 1
- net TAP1: track 0.00 -> 397.6 mm
- net TAP3: track 0.00 -> 361.2 mm, vias 0 -> 1
- net TAP5: track 0.00 -> 360.8 mm, vias 0 -> 1
- net TAP9: track 0.00 -> 358.8 mm, vias 0 -> 1
- net TAP7: track 0.00 -> 358.3 mm, vias 0 -> 1
- net TAP11: track 0.00 -> 354.4 mm, vias 0 -> 1
- net TAP13: track 0.00 -> 349.7 mm
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
Commit message: complete initial routing, layout, and silkscreen
Routing:
- net GND: track 80.4 -> 391.7 mm
- net +5V: track 75.3 -> 360.9 mm
- net TAP14: track 416.4 -> 409.5 mm
- net TAP0: track 442.8 -> 445.8 mm
Other:
- outline, holes or cut-outs redrawn
- board text added: "+"
- board text added: "+5V"
- board text added: "-"
- board text added: "0"
- board text added: "1"
- board text added: "10"
- board text added: "11"
- board text added: "12"
- board text added: "13"
- board text added: "14"
- board text added: "2"
- board text added: "3"
- board text added: "4"
- board text added: "5"
- board text added: "6"
- board text added: "7"
- board text added: "8"
- board text added: "9"
- board text added: "GND"
- board text added: "Modular Battery System 14S Backplane (Lite)"
- board text added: "r0 • Jun 2026 • Cy Westbrook"
